File: Hardware/SnapSerial Driver/SnapSerial Driver.kicad_sch (KiCad schematic)
At the start: 19 parts, among them J1 Power, J2 Conn_01x01_Pin, J3 M1, J4 M2, J5 PRT-14417, U1 ATtiny3217-M, U2 SPX3819M5-L-5-0, U3 A4950E, U4 A4950E

Commit message: Create Lumen and modify MF
Parts:
- R1: value R -> R0-220
Connections:
- net +5V renamed +V
Changed lines of the file:
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@@
 			)
 		)
-		(property "Value" "+5V"
+		(property "Value" "+V"
 			(at 87.122 67.818 0)
 			(effects
@@
 			)
 		)
-		(property "Value" "+5V"
+		(property "Value" "+V"
 			(at 107.442 50.546 90)
 			(effects
@@
 			)
 		)
-		(property "Value" "+5V"
-			(at 102.87 73.66 90)
+		(property "Value" "+V"
+			(at 102.87 73.66 0)
 			(effects
 				(font
@@
 		(on_board yes)
 		(dnp no)
-		(fields_autoplaced yes)
 		(property "Reference" "#PWR015"
 			(at 153.67 121.92 0)
@@
 			)
 		)
-		(property "Value" "+5V"
-			(at 146.05 121.92 90)
-			(effects
-				(font
-					(size 1.27 1.27)
-				)
-				(justify left)
+		(property "Value" "+V"
+			(at 145.796 124.714 90)
+			(effects
+				(font
+					(size 1.27 1.27)
+				)
+				(justify right)
 			)
 		)
@@
 			)
 		)
-		(property "Value" "+5V"
+		(property "Value" "+V"
 			(at 67.818 80.518 90)
 			(effects
@@
 			)
 		)
-		(property "Value" "+5V"
-			(at 128.27 49.53 90)
+		(property "Value" "+V"
+			(at 131.572 46.228 90)
 			(effects
 				(font
@@
 			)
 		)
-		(property "Value" "R"
+		(property "Value" "R0-220"
 			(at 52.07 77.47 90)
 			(effects
@@
 		(on_board yes)
 		(dnp no)
-		(fields_autoplaced yes)
 		(property "Reference" "#PWR014"
 			(at 153.67 91.44 0)
@@
 			)
 		)
-		(property "Value" "+5V"
-			(at 146.05 91.44 90)
-			(effects
-				(font
-					(size 1.27 1.27)
-				)
-				(justify left)
-			)
-		)
+		(property "Value" "+V"
+			(at 145.796 95.758 90)
+			(effects
+				(font
+					(size 1.27 1.27)
+				)
+				(justify right)
+			)
+		)
