File: Hardware/Lumen Daughterboard/Lumen.kicad_sch (KiCad schematic)
At the start: 14 parts, among them J5 PRT-14417, U1 ATtiny1617-M, U2 BNO055

Commit message: Update Lumen
Parts:
- added BZ1: Buzzer, User:CPT-9019A_CUD, symbol Device:Buzzer
- C1, C2, C3: footprint (none) -> Capacitor_SMD:C_0402_1005Metric
- D1, D2, D3, D4: footprint (none) -> LED_SMD:LED_0805_2012Metric
- J5: footprint User:CONN_PRT-14417_SPK -> User:QWIIC_SNAPSERIAL
- R1, R2, R3, R4: footprint (none) -> Resistor_SMD:R_0402_1005Metric
Connections:
- net GND: now also BZ1.2 (-)
- net at U1.5 (PA4): now also BZ1.1 (+)
- no-connect marks 16 -> 15
Other:
- moved on the sheet: J5
Changed lines of the file:
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@@
 		(at 130.81 43.18)
-	)
-	(no_connect
-		(at 130.81 50.8)
 	)
 	(wire
@@
 		(pts
 			(xy 137.16 99.06) (xy 143.51 99.06)
+		)
+		(stroke
+			(width 0)
+			(type default)
+		)
+	)
+	(wire
+		(pts
+			(xy 130.81 50.8) (xy 140.97 50.8)
 		)
 		(stroke
@@
 	)
 	(label "TX"
-		(at 90.17 27.94 270)
+		(at 157.48 29.21 270)
 		(effects
 			(font
@@
 	)
 	(label "RX"
-		(at 87.63 27.94 270)
+		(at 154.94 29.21 270)
 		(effects
 			(font
@@
 	(symbol
 		(lib_id "power:+5V")
-		(at 85.09 27.94 180)
+		(at 152.4 29.21 180)
 		(unit 1)
 		(exclude_from_sim no)
@@
 		(dnp no)
 		(property "Reference" "#PWR05"
-			(at 85.09 24.13 0)
+			(at 152.4 25.4 0)
 			(effects
 				(font
@@
 		)
 		(property "Value" "+V"
-			(at 85.852 32.258 0)
+			(at 153.162 33.528 0)
 			(effects
 				(font
@@
 		)
 		(property "Footprint" ""
-			(at 85.09 27.94 0)
+			(at 152.4 29.21 0)
 			(effects
 				(font
@@
 		)
 		(property "Datasheet" ""
-			(at 85.09 27.94 0)
+			(at 152.4 29.21 0)
 			(effects
 				(font
@@
 		)
 		(property "Description" ""
-			(at 85.09 27.94 0)
+			(at 152.4 29.21 0)
 			(effects
 				(font
@@
 	(symbol
 		(lib_id "New_Library:PRT-14417")
-		(at 82.55 27.94 90)
+		(at 149.86 29.21 90)
 		(unit 1)
 		(exclude_from_sim no)
@@
 		(fields_autoplaced yes)
 		(property "Reference" "J5"
-			(at 93.98 17.7799 90)
+			(at 161.29 19.0499 90)
 			(effects
 				(font
@@
 		)
 		(property "Value" "PRT-14417"
-			(at 93.98 20.3199 90)
+			(at 161.29 21.5899 90)
 			(effects
 				(font
@@
 			)
 		)
-		(property "Footprint" "User:CONN_PRT-14417_SPK"
-			(at 82.55 27.94 0)
+		(property "Footprint" "User:QWIIC_SNAPSERIAL"
+			(at 149.86 29.21 0)
 			(effects
 				(font
@@
 		)
 		(property "Datasheet" "PRT-14417"
-			(at 82.55 27.94 0)
+			(at 149.86 29.21 0)
 			(effects
 				(font
@@
 		)
 		(property "Description" ""
-			(at 82.55 27.94 0)
+			(at 149.86 29.21 0)
 			(effects
 				(font
@@
 			)
 		)
-		(property "Footprint" ""
+		(property "Footprint" "Resistor_SMD:R_0402_1005Metric"
 			(at 218.44 110.998 90)
 			(effects
@@
 			)
 		)
-		(property "Footprint" ""
+		(property "Footprint" "LED_SMD:LED_0805_2012Metric"
 			(at 130.81 95.25 0)
 			(effects
@@
 		(on_board yes)
 		(dnp no)
-		(fields_autoplaced yes)
 		(property "Reference" "D1"
-			(at 136.2075 50.8 0)
+			(at 137.922 59.944 0)
 			(effects
 				(font
@@
 		)
 		(property "Value" "LED"
-			(at 136.2075 53.34 0)
-			(effects
-				(font
-					(size 1.27 1.27)
-				)
-			)
-		)
-		(property "Footprint" ""
+			(at 137.922 62.484 0)
+			(effects
+				(font
+					(size 1.27 1.27)
+				)
+			)
+		)
+		(property "Footprint" "LED_SMD:LED_0805_2012Metric"
 			(at 134.62 58.42 0)
 			(effects
@@
 			)
 		)
-		(property "Footprint" ""
+		(property "Footprint" "Resistor_SMD:R_0402_1005Metric"
 			(at 218.44 107.188 90)
 			(effects
@@
 			)
 		)
-		(property "Footprint" ""
+		(property "Footprint" "Capacitor_SMD:C_0402_1005Metric"
 			(at 115.57 30.7848 0)
 			(effects
@@
 			)
 		)
-		(property "Footprint" ""
+		(property "Footprint" "Capacitor_SMD:C_0402_1005Metric"
 			(at 191.77 84.7852 0)
 			(effects
@@
 	)
 	(symbol
+		(lib_id "power:GND")
+		(at 146.05 50.8 90)
+		(unit 1)
+		(exclude_from_sim no)
+		(in_bom yes)
+		(on_board yes)
+		(dnp no)
+		(fields_autoplaced yes)
+		(property "Reference" "#PWR017"
+			(at 152.4 50.8 0)
+			(effects
+				(font
+					(size 1.27 1.27)
+				)
+				(hide yes)
+			)
+		)
+		(property "Value" "GND"
+			(at 149.86 50.7999 90)
+			(effects
+				(font
+					(size 1.27 1.27)
+				)
+				(justify right)
+			)
+		)
+		(property "Footprint" ""
+			(at 146.05 50.8 0)
+			(effects
+				(font
+					(size 1.27 1.27)
+				)
+				(hide yes)
+			)
+		)
+		(property "Datasheet" ""
+			(at 146.05 50.8 0)
+			(effects
+				(font
+					(size 1.27 1.27)
+				)
+				(hide yes)
+			)
+		)
+		(property "Description" "Power symbol creates a global label with name \"GND\" , ground"
+			(at 146.05 50.8 0)
+			(effects
+				(font
+					(size 1.27 1.27)
+				)
+				(hide yes)
+			)
+		)
+		(pin "1"
+		)
+		(instances
+			(project "Lumen"
+				(path "/6b836b10-3dda-47fa-ae17-1c3cd42ae45d"
+					(reference "#PWR017")
+					(unit 1)
+				)
+			)
+		)
+	)
+	(symbol
 		(lib_id "Device:R")
 		(at 157.48 83.82 270)
@@
 			)
 		)
-		(property "Footprint" ""
+		(property "Footprint" "Resistor_SMD:R_0402_1005Metric"
 			(at 157.48 82.042 90)
 			(effects
@@
 			)
 		)
-		(property "Footprint" ""
+		(property "Footprint" "LED_SMD:LED_0805_2012Metric"
 			(at 137.16 95.25 0)
 			(effects
@@
 			)
 		)
-		(property "Footprint" ""
+		(property "Footprint" "LED_SMD:LED_0805_2012Metric"
 			(at 143.51 95.25 0)
 			(effects
@@
 	(symbol
 		(lib_id "power:GND")
-		(at 82.55 27.94 0)
+		(at 149.86 29.21 0)
 		(unit 1)
 		(exclude_from_sim no)
@@
 		(dnp no)
 		(property "Reference" "#PWR04"
-			(at 82.55 34.29 0)
+			(at 149.86 35.56 0)
 			(effects
 				(font
@@
 		)
 		(property "Value" "GND"
-			(at 78.232 31.242 0)
+			(at 145.542 32.512 0)
 			(effects
 				(font
@@
 		)
 		(property "Footprint" ""
-			(at 82.55 27.94 0)
+			(at 149.86 29.21 0)
 			(effects
 				(font
@@
 		)
 		(property "Datasheet" ""
-			(at 82.55 27.94 0)
+			(at 149.86 29.21 0)
 			(effects
 				(font
@@
 		)
 		(property "Description" ""
-			(at 82.55 27.94 0)
+			(at 149.86 29.21 0)
 			(effects
 				(font
@@
 			)
 		)
-		(property "Footprint" ""
+		(property "Footprint" "Capacitor_SMD:C_0402_1005Metric"
 			(at 173.99 49.8348 0)
 			(effects
@@
 			)
 		)
-		(property "Footprint" ""
+		(property "Footprint" "Resistor_SMD:R_0402_1005Metric"
 			(at 218.44 103.378 90)
 			(effects
@@
 					(unit 1)
 				)
+			)
+		)
+	)
+	(symbol
+		(lib_id "Device:Buzzer")
+		(at 143.51 48.26 90)
+		(unit 1)
+		(exclude_from_sim no)
+		(in_bom yes)
+		(on_board yes)
+		(dnp no)
+		(fields_autoplaced yes)
+		(property "Reference" "BZ1"
+			(at 147.32 46.2348 90)
+			(effects
+				(font
+					(size 1.27 1.27)
+				)
+				(justify right)
+			)
+		)
+		(property "Value" "Buzzer"
+			(at 147.32 48.7748 90)
+			(effects
+				(font
+					(size 1.27 1.27)
+				)
+				(justify right)
+			)
+		)
+		(property "Footprint" "User:CPT-9019A_CUD"
+			(at 140.97 48.895 90)
+			(effects
+				(font
+					(size 1.27 1.27)
+				)
+				(hide yes)
+			)
+		)
+		(property "Datasheet" "~"
+			(at 140.97 48.895 90)
+			(effects
+				(font
+					(size 1.27 1.27)
+				)
+				(hide yes)
+			)
+		)
+		(property "Description" "Buzzer, polarized"
+			(at 143.51 48.26 0)
+			(effects
+				(font
+					(size 1.27 1.27)
+				)
+				(hide yes)
+			)
+		)
+		(pin "1"
+		)
+		(pin "2"
+		)
+		(instances
+			(project ""
+				(path "/6b836b10-3dda-47fa-ae17-1c3cd42ae45d"
+					(reference "BZ1")
+					(unit 1)
+				)

Commit message: Lumen :D
Parts:
- removed BZ1: Buzzer, User:CPT-9019A_CUD, symbol Device:Buzzer
- added J1: Conn_01x01_Socket, Connector_PinSocket_2.54mm:PinSocket_1x01_P2.54mm_Vertical, symbol Connector:Conn_01x01_Socket
Connections:
- net UPDI: now also J1.1 (Pin_1)
- no-connect marks 15 -> 16
Changed lines of the file:
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@@
+	)
+	(no_connect
+		(at 130.81 50.8)
 	)
 	(no_connect
@@
 		(pts
 			(xy 137.16 99.06) (xy 143.51 99.06)
-		)
-		(stroke
-			(width 0)
-			(type default)
-		)
-	)
-	(wire
-		(pts
-			(xy 130.81 50.8) (xy 140.97 50.8)
 		)
 		(stroke
@@
 		)
 	)
+	(label "UPDI"
+		(at 120.65 24.13 270)
+		(effects
+			(font
+				(size 1.27 1.27)
+			)
+			(justify right bottom)
+		)
+	)
 	(label "TX"
 		(at 157.48 29.21 270)
@@
 	)
 	(symbol
-		(lib_id "power:GND")
-		(at 146.05 50.8 90)
-		(unit 1)
-		(exclude_from_sim no)
-		(in_bom yes)
-		(on_board yes)
-		(dnp no)
-		(fields_autoplaced yes)
-		(property "Reference" "#PWR017"
-			(at 152.4 50.8 0)
-			(effects
-				(font
-					(size 1.27 1.27)
-				)
-				(hide yes)
-			)
-		)
-		(property "Value" "GND"
-			(at 149.86 50.7999 90)
-			(effects
-				(font
-					(size 1.27 1.27)
-				)
-				(justify right)
-			)
-		)
-		(property "Footprint" ""
-			(at 146.05 50.8 0)
-			(effects
-				(font
-					(size 1.27 1.27)
-				)
-				(hide yes)
-			)
-		)
-		(property "Datasheet" ""
-			(at 146.05 50.8 0)
-			(effects
-				(font
-					(size 1.27 1.27)
-				)
-				(hide yes)
-			)
-		)
-		(property "Description" "Power symbol creates a global label with name \"GND\" , ground"
-			(at 146.05 50.8 0)
-			(effects
-				(font
-					(size 1.27 1.27)
-				)
-				(hide yes)
-			)
-		)
-		(pin "1"
-		)
-		(instances
-			(project "Lumen"
-				(path "/6b836b10-3dda-47fa-ae17-1c3cd42ae45d"
-					(reference "#PWR017")
-					(unit 1)
-				)
-			)
-		)
-	)
-	(symbol
 		(lib_id "Device:R")
 		(at 157.48 83.82 270)
@@
 	)
 	(symbol
+		(lib_id "Connector:Conn_01x01_Socket")
+		(at 120.65 19.05 90)
+		(unit 1)
+		(exclude_from_sim no)
+		(in_bom yes)
+		(on_board yes)
+		(dnp no)
+		(fields_autoplaced yes)
+		(property "Reference" "J1"
+			(at 121.92 18.4149 90)
+			(effects
+				(font
+					(size 1.27 1.27)
+				)
+				(justify right)
+			)
+		)
+		(property "Value" "Conn_01x01_Socket"
+			(at 121.92 20.9549 90)
+			(effects
+				(font
+					(size 1.27 1.27)
+				)
+				(justify right)
+			)
+		)
+		(property "Footprint" "Connector_PinSocket_2.54mm:PinSocket_1x01_P2.54mm_Vertical"
+			(at 120.65 19.05 0)
+			(effects
+				(font
+					(size 1.27 1.27)
+				)
+				(hide yes)
+			)
+		)
+		(property "Datasheet" "~"
+			(at 120.65 19.05 0)
+			(effects
+				(font
+					(size 1.27 1.27)
+				)
+				(hide yes)
+			)
+		)
+		(property "Description" "Generic connector, single row, 01x01, script generated"
+			(at 120.65 19.05 0)
+			(effects
+				(font
+					(size 1.27 1.27)
+				)
+				(hide yes)
+			)
+		)
+		(pin "1"
+		)
+		(instances
+			(project ""
+				(path "/6b836b10-3dda-47fa-ae17-1c3cd42ae45d"
+					(reference "J1")
+					(unit 1)
+				)
+			)
+		)
+	)
+	(symbol
 		(lib_id "MCU_Microchip_ATtiny:ATtiny1617-M")
 		(at 115.57 60.96 0)
@@
 					(unit 1)
 				)
-			)
-		)
-	)
-	(symbol
-		(lib_id "Device:Buzzer")
-		(at 143.51 48.26 90)
-		(unit 1)
-		(exclude_from_sim no)
-		(in_bom yes)
-		(on_board yes)
-		(dnp no)
-		(fields_autoplaced yes)
-		(property "Reference" "BZ1"
-			(at 147.32 46.2348 90)
-			(effects
-				(font
-					(size 1.27 1.27)
-				)
-				(justify right)
-			)
-		)
-		(property "Value" "Buzzer"
-			(at 147.32 48.7748 90)
-			(effects
-				(font
-					(size 1.27 1.27)
-				)
-				(justify right)
-			)
-		)
-		(property "Footprint" "User:CPT-9019A_CUD"
-			(at 140.97 48.895 90)
-			(effects
-				(font
-					(size 1.27 1.27)
-				)
-				(hide yes)
-			)
-		)
-		(property "Datasheet" "~"
-			(at 140.97 48.895 90)
-			(effects
-				(font
-					(size 1.27 1.27)
-				)
-				(hide yes)
-			)
-		)
-		(property "Description" "Buzzer, polarized"
-			(at 143.51 48.26 0)
-			(effects
-				(font
-					(size 1.27 1.27)
-				)
-				(hide yes)
-			)
-		)
-		(pin "1"
-		)
-		(pin "2"
-		)
-		(instances
-			(project ""
-				(path "/6b836b10-3dda-47fa-ae17-1c3cd42ae45d"
-					(reference "BZ1")
-					(unit 1)
-				)
