File: Impulse/Kicad/Impulse Driver.kicad_pcb (KiCad board)
At the start: 2 copper layers, 14.2 x 22 mm, 26 parts, among them J1 Power, J2 UPDI, J3 M1, J4 M2, J5 PRT-14417, U1 ATtiny1617-M, U3 A4950E, U4 A4950E

Commit message: fix severe error with low current 12v lines
Parts:
- U2: value ~ -> TPS56124
- moved D2 2.16 mm to (151.0, 103.5), turned to 90 degrees
Connections:
- C1 pad 1: Net-(D2-A) -> +BATT
- C12 pad 2: +BATT -> Net-(D2-K)
- D2 pad 1: +BATT -> Net-(D2-K)
- D2 pad 2: Net-(D2-A) -> +BATT
- J1 pad 1: Net-(D2-A) -> +BATT
- R8 pad 2: +BATT -> Net-(D2-K)
- U2 pad 1: +BATT -> Net-(D2-K)
Routing:
- net Net-(D2-K): track 0.00 -> 14.2 mm, vias 0 -> 2
- net +BATT: track 35.0 -> 22.6 mm, vias 4 -> 3
- net Net-(D2-A): track 1.97 -> 0.00 mm, vias 1 -> 0
Other:
- board text added: "R4 Impulse"
- board text removed: "R3 Impulse"

Commit message: update impulse to r5
Parts:
- removed C10: 22uF, Capacitor_SMD:C_0805_2012Metric
- removed C11, C12: 0.1uF, Capacitor_SMD:C_0402_1005Metric
- removed C9: 47pF, Capacitor_SMD:C_0402_1005Metric
- removed D2: 1.5A, Diode_SMD:D_SOD-123F
- removed L2: 3.3uH, Inductor_SMD:L_Changjiang_FTC201610S
- removed R5: 30k, Resistor_SMD:R_0402_1005Metric
- removed R8: 100k, Resistor_SMD:R_0402_1005Metric
- added C5: 10uF, Capacitor_SMD:C_0805_2012Metric, F.Cu at (148.9, 104.7)
- added C6: 22uF, Capacitor_SMD:C_0805_2012Metric, F.Cu at (151.9, 107.0)
- added L1: 2.2uH 48mOhm, Inductor_SMD:L_Pulse_PA4332, F.Cu at (150.7, 111.3)
- R4: value 135k -> 100k; moved to B.Cu
- U1: value ATtiny1617-M -> ATtiny3217-M
- U2: value TPS56124 -> TPS62162DSG; footprint Package_TO_SOT_SMD:SOT-563 -> Package_SON:Texas_DSG0008A_WSON-8-1EP_2x2mm_P0.5mm_EP0.9x1.6mm_ThermalVias
- moved R4 9.25 mm to (154.6, 106.8), turned to -90 degrees
- moved J5 5.68 mm to (144.7, 111.6)
- moved C4 4.57 mm to (144.3, 112.9), turned to 180 degrees
- moved U2 3.33 mm to (148.9, 107.2), turned to -90 degrees
- moved J2 0.93 mm to (143.3, 105.8)
- moved U1 0.57 mm to (145.0, 109.8), turned to 90 degrees
- moved J1 0.15 mm to (153.8, 102.0)
Connections:
- R4 pad 2: Net-(U2-FB) -> Net-(U2-PG)
- U1 pad 15: unconnected-(U1-PB1-Pad15) -> /M2_IN1
- U1 pad 16: unconnected-(U1-PB0-Pad16) -> /M2_IN2
- U1 pad 19: /M2_IN1 -> unconnected-(U1-PC2-Pad19)
- U1 pad 20: /M2_IN2 -> unconnected-(U1-PC3-Pad20)
- U1 pad 21: /M1_IN1 -> unconnected-(U1-PC4-Pad21)
- U1 pad 22: /M1_IN2 -> unconnected-(U1-PC5-Pad22)
- U1 pad 5: unconnected-(U1-PA4-Pad5) -> /M1_IN1
- U1 pad 6: unconnected-(U1-PA5-Pad6) -> /M1_IN2
- U2 pad 1: Net-(D2-K) -> GND
- U2 pad 2: Net-(U2-SW) -> +BATT
- U2 pad 3: GND -> +BATT
- U2 pad 4: Net-(U2-BST) -> GND
- U2 pad 5: Net-(U2-EN) -> GND
- U2 pad 6: Net-(U2-FB) -> +3V3
Routing:
- net GND: track 12.9 -> 29.1 mm, vias 9 -> 8
- net /M1_IN2: track 5.71 -> 20.0 mm
- net Net-(D2-K): track 14.2 -> 0.00 mm, vias 2 -> 0
- net /M1_IN1: track 6.28 -> 19.5 mm
- net +3V3: track 11.5 -> 22.3 mm, vias 7 -> 5
- net Net-(U2-PG): track 0.00 -> 5.84 mm, vias 0 -> 1
- net Net-(U2-FB): track 4.28 -> 0.00 mm
- net /TX: track 2.35 -> 6.22 mm
- net Net-(J2-Pin_1): track 3.13 -> 6.01 mm, vias 1 -> 0
- net Net-(U2-SW): track 5.43 -> 3.10 mm
- net /M2_IN2: track 6.48 -> 8.80 mm
- net /RX: track 3.88 -> 5.37 mm
- net /M2_IN1: track 7.73 -> 9.12 mm
- net Net-(U2-EN): track 1.12 -> 0.00 mm
- net Net-(U2-BST): track 1.04 -> 0.00 mm
- added copper zone on B.Cu, net +BATT
- added copper zone on F.Cu, net +BATT
Other:
- board text added: "R5 Impulse"
- board text removed: "M1"
- board text removed: "M2"
- board text removed: "R4 Impulse"
- board text removed: "Snap"
- board text removed: "UPDI"
