File: Impulse/Kicad/Impulse Driver.kicad_sch (KiCad schematic)
At the start: 26 parts, among them J1 Power, J2 UPDI, J3 M1, J4 M2, J5 PRT-14417, U1 ATtiny1617-M, U3 A4950E, U4 A4950E

Commit message: work on the impulse bom
Parts:
- C1: LCSC (none) -> C440198
- C10: LCSC (none) -> C602037
- C11, C12, C2, C3, C4: LCSC (none) -> C14663
- C9: LCSC (none) -> C60137
- D1: LCSC (none) -> C965814
- R1: LCSC (none) -> C2909336
- R2, R3: LCSC (none) -> C7467478
- R4: LCSC (none) -> C2515705
- R5: LCSC (none) -> C2909347
- R8: LCSC (none) -> C25741
- U1: LCSC (none) -> C1340514
- U2: value (none) -> TPS56124
- U3, U4: LCSC (none) -> C82404

Commit message: fix severe error with low current 12v lines
Connections:
- net +BATT: now also C1.1, D2.2 (A), J1.1 (Pin_1); no longer C12.2, D2.1 (K), R8.2, U2.1 (VIN)
- new net: C12.2, D2.1 (K), R8.2, U2.1 (VIN)

Commit message: update impulse to r5
Parts:
- removed C10: 22uF, Capacitor_SMD:C_0805_2012Metric, symbol Device:C_Small
- removed C11, C12: 0.1uF, Capacitor_SMD:C_0402_1005Metric, symbol Device:C_Small
- removed C9: 47pF, Capacitor_SMD:C_0402_1005Metric, symbol Device:C_Small
- removed D2: 1.5A, Diode_SMD:D_SOD-123F, symbol Device:D_Small
- removed L2: 3.3uH, Inductor_SMD:L_Changjiang_FTC201610S, symbol Device:L_Small
- removed R5: 30k, Resistor_SMD:R_0402_1005Metric, symbol Device:R_Small
- removed R8: 100k, Resistor_SMD:R_0402_1005Metric, symbol Device:R_Small
- removed U2: TPS56124, Package_TO_SOT_SMD:SOT-563, symbol Impulse Driver:TPS561246
- added C5: 10uF, Capacitor_SMD:C_0805_2012Metric, symbol Device:C_Small
- added C6: 22uF, Capacitor_SMD:C_0805_2012Metric, symbol Device:C_Small
- added L1: 2.2uH 48mOhm, Inductor_SMD:L_Pulse_PA4332, symbol Device:L_Small
- added U2: TPS62162DSG, Package_SON:Texas_DSG0008A_WSON-8-1EP_2x2mm_P0.5mm_EP0.9x1.6mm_ThermalVias, symbol Regulator_Switching:TPS62162DSG
- R4: value 135k -> 100k; LCSC C2515705 -> (none)
- U1: value ATtiny1617-M -> ATtiny3217-M; symbol MCU_Microchip_ATtiny:ATtiny1617-M -> MCU_Microchip_ATtiny:ATtiny3217-M
Connections:
- net +3V3: now also C6.1, L1.2, U2.6 (VOS)
- net +BATT: now also C5.1, U2.2 (VIN), U2.3 (EN)
- net GND: now also C5.2, C6.2, U2.1 (PGND), U2.4 (AGND), U2.5 (FB), U2.9 (PAD)
- net M1_IN1: now also U1.5 (PA4); no longer U1.21 (PC4)
- net M1_IN2: now also U1.6 (PA5); no longer U1.22 (PC5)
- net M2_IN1: now also U1.15 (PB1); no longer U1.19 (PC2)
- net M2_IN2: now also U1.16 (PB0); no longer U1.20 (PC3)
- net at R4.2: now also U2.8 (PG)
- new net: L1.1, U2.7 (SW)
- no-connect marks 1 -> 15
